Commit message: udpate gripper

File: urdf/gripper_robot.urdf (robot description, URDF)
Before this commit: robot gripper_robot, 8 links, 7 joints
Links:
- link link4: geometry collision cylinder length=0.4 radius=0.05; visual cylinder length=0.4 radius=0.05
- link link5: geometry collision box size=0.1 0.1 0.4; visual box size=0.1 0.1 0.4
- link link6: geometry collision box size=0.1 0.1 0.4; visual box size=0.1 0.1 0.4
